File: docs/v3-adder.kicad_sch (KiCad schematic)
At the start: 102 parts, among them J1 Thonkiconn, J2 Thonkiconn, J3 Thonkiconn, J4 Thonkiconn, J5 Thonkiconn, J6 Thonkiconn, J7 Thonkiconn, J8 Thonkiconn, P1 Eurorack 2x5, SW1A SUBMINI ON-OFF-ON, SW1B SUBMINI ON-ON, SW2A SUBMINI ON-OFF-ON, SW2B SUBMINI ON-ON-ON, SW3A SUBMINI ON-OFF-ON, SW3B SUBMINI ON-ON-ON, SW4A SUBMINI ON-OFF-ON, SW4B SUBMINI ON-ON-ON, U1 OPA4196, U2 OPA4196, U3 OPA4196, U4 L78L05, U5 L79L05

Commit message: Schematic: fix unresolved symbols, draw real bodies
Every symbol rendered as a box with "??" - KiCad's missing-symbol placeholder.
lib_symbols entries must be named with the full LIBRARY:NAME, and they were
named bare ("R" where instances referenced "adder:R"), so nothing resolved.

The check that should have caught this could not: it compared
libId.split(':')[-1] on both sides, stripping the very prefix that was wrong.
It now compares whole lib_id strings, and additionally confirms each
instantiated unit has a matching body, and that all 267 pin coordinates read
back out of the written file land on a wire endpoint - so the label stubs are
attached to pins rather than merely near them.

Bodies were placeholder rectangles, so they are now drawn properly: diode with
the bar on the cathode end, switches with a lever from common to a throw,
trimmer with a wiper arrow, jack with sleeve and tip contacts, ferrite, and the
power header as the physical 2x5 with odd pins left and even pins right. Two-pin
passives hide pin names and numbers, as the stock KiCad symbols do.

Co-Authored-By: Claude Opus 5 <noreply@anthropic.com>
Connections:
- net +12V: now also C1.1, C2.1, C5.1, D1.1 (K), U1.4 (V+), U2.4 (V+), U3.4 (V+), U4.1 (IN)
- net +5V: now also C6.1, R1.1, U4.3 (OUT)
- net -12V: now also C3.1, C4.1, C7.1, D2.2 (A), U1.11 (V-), U2.11 (V-), U3.11 (V-), U5.1 (IN)
- net -5V: now also C8.1, R3.1, U5.3 (OUT)
- net BIAS1: now also C11.1, R17.1, R18.2, R19.1, R19.2, U1.10 (+), U1.6 (-), U1.7
- net BIAS1_SEL: now also C11.2, SW1B.2 (COM), U1.5 (+)
- net BIAS1_SNUB: now also C12.1, R17.2
- net BIAS2: now also C13.1, R27.1, R28.2, R29.1, R29.2, U1.13 (-), U1.14, U2.3 (+)
- net BIAS2_SEL: now also C13.2, SW2B.4 (COM), U1.12 (+)
- net BIAS2_SNUB: now also C14.1, R27.2
- net BIAS3: now also C15.1, R37.1, R38.2, R39.1, R39.2, U2.10 (+), U2.6 (-), U2.7
- net BIAS3_SEL: now also C15.2, SW3B.4 (COM), U2.5 (+)
- net BIAS3_SNUB: now also C16.1, R37.2
- net BIAS4: now also C17.1, R47.1, R48.2, R49.1, R49.2, U2.13 (-), U2.14, U3.3 (+)
- net BIAS4_SEL: now also C17.2, SW4B.4 (COM), U2.12 (+)
- net BIAS4_SNUB: now also C18.1, R47.2
- net FB1: now also R20.2, R21.1, U1.9 (-)
- net FB2: now also R30.2, R31.1, U2.2 (-)
- net FB3: now also R40.2, R41.1, U2.9 (-)
- net FB4: now also R50.2, R51.1, U3.2 (-)
- net GND: now also C1.2, C10.2, C12.2, C14.2, C16.2, C18.2, C2.2, C3.2, C4.2, C5.2, C6.2, C7.2, C8.2, C9.2, J1.2 (S), J2.2 (S), J3.2 (S), J4.2 (S), J5.2 (S), J6.2 (S), J7.2 (S), J8.2 (S), P1.3 (P3), P1.4 (P4), P1.5 (P5), P1.6 (P6), P1.7 (P7), P1.8 (P8), R12.2, R14.1, R2.2, R21.2, R23.1, R31.2, R33.1, R4.2, R41.2, R43.1, R5.2, R51.2, R7.2, R9.2, U3.5 (+), U4.2 (GND), U5.2 (GND)
- net IN1: now also J1.1 (T), R5.1, R6.1
- net IN2: now also J2.1 (T), R7.1, R8.1
- net IN3: now also J3.1 (T), R10.1, R9.1
- net LAD1_TOP: now also SW1A.2 (COM), VR1.1
- net LAD1_TRIM: now also R16.2, VR1.2 (W), VR1.3
- net LAD2_TOP: now also SW2A.2 (COM), VR2.1
- net LAD2_TRIM: now also R26.2, VR2.2 (W), VR2.3
- net LAD3_TOP: now also SW3A.2 (COM), VR3.1
- net LAD3_TRIM: now also R36.2, VR3.2 (W), VR3.3
- net LAD4_TOP: now also SW4A.2 (COM), VR4.1
- net LAD4_TRIM: now also R46.2, VR4.2 (W), VR4.3
- net N12_F: now also D2.1 (K), FB2.2
- net N12_RAW: now also FB2.1, P1.1 (P1), P1.2 (P2)
- net OCT_1V: now also R14.2, R15.1, SW1B.1 (A)
- net OCT_2V: now also R15.2, R16.1, SW1B.3 (B)
- net OUT1: now also R20.1, R22.1, R28.1, U1.8
- net OUT1_JACK: now also J5.1 (T), R22.2
- net OUT2: now also R30.1, R32.1, R38.1, U2.1
- net OUT2_JACK: now also J6.1 (T), R32.2
- net OUT3: now also R40.1, R42.1, R48.1, U2.8
- net OUT3_JACK: now also J7.1 (T), R42.2
- net OUT4: now also R50.1, R52.1, U3.1
- net OUT4_JACK: now also J8.1 (T), R52.2
- net P12_F: now also D1.2 (A), FB1.2
- net P12_RAW: now also FB1.1, P1.10 (P10), P1.9 (P9)
- net REFN_BOT: now also R4.1, VR6.3
- net REFN_TOP: now also R3.2, VR6.1
- net REFN_W: now also U3.12 (+), VR6.2 (W)
- net REFP_BOT: now also R2.1, VR5.3
- net REFP_TOP: now also R1.2, VR5.1
- net REFP_W: now also U3.10 (+), VR5.2 (W)
- net S2_4th: now also R25.2, R26.1, SW2B.1 (A)
- net S2_M3: now also R24.2, R25.1, SW2B.2 (B)
- net S2_m3: now also R23.2, R24.1, SW2B.3 (C)
- net S3_4th: now also R35.2, R36.1, SW3B.1 (A)
- net S3_M3: now also R34.2, R35.1, SW3B.2 (B)
- net S3_m3: now also R33.2, R34.1, SW3B.3 (C)
- net S4_5th: now also R45.2, R46.1, SW4B.1 (A)
- net S4_M3: now also R44.2, R45.1, SW4B.2 (B)
- net S4_m3: now also R43.2, R44.1, SW4B.3 (C)
- net SUMFB: now also R11.2, R12.1, U1.2 (-)
- net SUMNODE: now also R10.2, R6.2, R8.2, U1.3 (+)
- net SUM_BUS: now also R11.1, R13.1, R18.1, U1.1
- net SUM_JACK: now also J4.1 (T), R13.2
- net U3B_OUT: now also U3.6 (-), U3.7
- net VREF_N: now also C10.1, SW1A.3 (B), SW2A.3 (B), SW3A.3 (B), SW4A.3 (B), U3.13 (-), U3.14
- net VREF_P: now also C9.1, SW1A.1 (A), SW2A.1 (A), SW3A.1 (A), SW4A.1 (A), U3.8, U3.9 (-)
Changed lines of the file:
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@@
     (property "Datasheet" "~" (at 40 60 0) (effects (font (size 1.27 1.27)) hide))
     (pin "1")
-    (pin "2")
-    (pin "3")
+    (pin "3")
+    (pin "5")
+    (pin "7")
+    (pin "9")
+    (pin "2")
     (pin "4")
-    (pin "5")
     (pin "6")
-    (pin "7")
     (pin "8")
-    (pin "9")
     (pin "10")
     (instances
@@
     )
   )
-  (wire (pts (xy 34.92 49.84) (xy 31.110000000000003 49.84)) (stroke (width 0) (type default)))
-  (label "N12_RAW" (at 31.110000000000003 49.84 180) (effects (font (size 1.0 1.0))))
-  (wire (pts (xy 34.92 52.38) (xy 31.110000000000003 52.38)) (stroke (width 0) (type default)))
-  (label "N12_RAW" (at 31.110000000000003 52.38 180) (effects (font (size 1.0 1.0))))
   (wire (pts (xy 34.92 54.92) (xy 31.110000000000003 54.92)) (stroke (width 0) (type default)))
-  (label "GND" (at 31.110000000000003 54.92 180) (effects (font (size 1.0 1.0))))
+  (label "N12_RAW" (at 31.110000000000003 54.92 180) (effects (font (size 1.0 1.0))))
   (wire (pts (xy 34.92 57.46) (xy 31.110000000000003 57.46)) (stroke (width 0) (type default)))
   (label "GND" (at 31.110000000000003 57.46 180) (effects (font (size 1.0 1.0))))
@@
   (label "GND" (at 31.110000000000003 62.54 180) (effects (font (size 1.0 1.0))))
   (wire (pts (xy 34.92 65.08) (xy 31.110000000000003 65.08)) (stroke (width 0) (type default)))
-  (label "GND" (at 31.110000000000003 65.08 180) (effects (font (size 1.0 1.0))))
-  (wire (pts (xy 34.92 67.62) (xy 31.110000000000003 67.62)) (stroke (width 0) (type default)))
-  (label "GND" (at 31.110000000000003 67.62 180) (effects (font (size 1.0 1.0))))
-  (wire (pts (xy 34.92 70.16) (xy 31.110000000000003 70.16)) (stroke (width 0) (type default)))
-  (label "P12_RAW" (at 31.110000000000003 70.16 180) (effects (font (size 1.0 1.0))))
-  (wire (pts (xy 34.92 72.7) (xy 31.110000000000003 72.7)) (stroke (width 0) (type default)))
-  (label "P12_RAW" (at 31.110000000000003 72.7 180) (effects (font (size 1.0 1.0))))
+  (label "P12_RAW" (at 31.110000000000003 65.08 180) (effects (font (size 1.0 1.0))))
+  (wire (pts (xy 45.08 54.92) (xy 48.89 54.92)) (stroke (width 0) (type default)))
+  (label "N12_RAW" (at 48.89 54.92 0) (effects (font (size 1.0 1.0))))
+  (wire (pts (xy 45.08 57.46) (xy 48.89 57.46)) (stroke (width 0) (type default)))
+  (label "GND" (at 48.89 57.46 0) (effects (font (size 1.0 1.0))))
+  (wire (pts (xy 45.08 60.0) (xy 48.89 60.0)) (stroke (width 0) (type default)))
+  (label "GND" (at 48.89 60.0 0) (effects (font (size 1.0 1.0))))
+  (wire (pts (xy 45.08 62.54) (xy 48.89 62.54)) (stroke (width 0) (type default)))
+  (label "GND" (at 48.89 62.54 0) (effects (font (size 1.0 1.0))))
+  (wire (pts (xy 45.08 65.08) (xy 48.89 65.08)) (stroke (width 0) (type default)))
+  (label "P12_RAW" (at 48.89 65.08 0) (effects (font (size 1.0 1.0))))
   (wire (pts (xy 64.92 40) (xy 61.11 40.0)) (stroke (width 0) (type default)))
   (label "P12_RAW" (at 61.11 40.0 180) (effects (font (size 1.0 1.0))))

Commit message: Schematic: ERC-clean, and run KiCad's own checks
KiCad 7 and 10 are installed on this machine; kicad-cli runs from WSL against
the Windows binary, so ERC and DRC are no longer things I could only promise to
someone else. tools/kicad-check.sh runs both and plots both.

ERC went 553 violations to 23, and 3 errors to 0. What it caught:

- BIAS and SUM were SHORTED on every stage. Two 10k resistors sat 12 mm apart
  but each occupies +/-7.62 mm with its label stubs, so the stubs overlapped
  and tied the bias buffer straight past its summing resistor. My checks could
  not see it: I verify the netlist I declare, KiCad computes connectivity from
  geometry. Parts are now placed one per cell on a 25.4 mm lattice, wide enough
  for the largest symbol plus stubs, so stubs cannot touch.
- 381 off-grid endpoints, from hand-picked coordinates that were not multiples
  of 1.27. The lattice fixes these too - 25.4 is 20 x 1.27.
- S2_m3 vs S2_M3 differed only in case. Renamed MIN3 / MAJ3.
- +12V, -12V and GND had no power-output driving them; added PWR_FLAG symbols.

The rest was library noise, now dealt with: the generator also writes
adder.kicad_sym, v3-adder.kicad_pro and a sym-lib-table so the project opens
with its symbols resolved, and footprints point at stock KiCad libraries
wherever they exist. The 23 that remain are footprint links on the custom parts
- jacks, toggles, trimmers, ferrites, power header - which are the user's to
supply.

The panel passes DRC with 0 violations and 0 unconnected items, and plots
correctly from KiCad, which also confirms the obround mounting slots in KiCad's
own renderer rather than only in my SVG preview.

Co-Authored-By: Claude Opus 5 <noreply@anthropic.com>
Parts:
- C1, C10, C3, C9: footprint (none) -> Capacitor_THT:CP_Radial_D5.0mm_P2.00mm
- C11, C12, C13, C14, C15, C16, C17, C18, C2, C4, C5, C6, C7, C8: footprint (none) -> Capacitor_SMD:C_0805_2012Metric
- D1, D2: footprint DO-41 -> Diode_THT:D_DO-41_SOD81_P10.16mm_Horizontal
- R1, R10, R11, R12, R13, R14, R15, R16, R17, R18, R19, R2, R20, R21, R22, R23, R24, R25, R26, R27, R28, R29, R3, R30, R31, R32, R33, R34, R35, R36, R37, R38, R39, R4, R40, R41, R42, R43, R44, R45, R46, R47, R48, R49, R5, R50, R51, R52, R6, R7, R8, R9: footprint (none) -> Resistor_SMD:R_0805_2012Metric
- U1, U2, U3: footprint (none) -> Package_SO:SOIC-14_3.9x8.7mm_P1.27mm
- U1, U2, U3: footprint SOIC-14_150MIL -> Package_SO:SOIC-14_3.9x8.7mm_P1.27mm
- U4, U5: footprint TO-92-3_L4.8-W3.7-P2.54-L -> Package_TO_SOT_THT:TO-92_Inline
Connections:
- net BIAS1: no longer R18.2, R19.2, U1.10 (+)
- net BIAS2: no longer R28.2, R29.2, U2.3 (+)
- net BIAS3: no longer R38.2, R39.2, U2.10 (+)
- net BIAS4: no longer R48.2, R49.2, U3.3 (+)
- net S2_M3 renamed S2_MAJ3
- net S2_m3 renamed S2_MIN3
- net S3_M3 renamed S3_MAJ3
- net S3_m3 renamed S3_MIN3
- net S4_M3 renamed S4_MAJ3
- net S4_m3 renamed S4_MIN3
- new net SUM1: R18.2, R19.2, U1.10 (+)
- new net SUM2: R28.2, R29.2, U2.3 (+)
- new net SUM3: R38.2, R39.2, U2.10 (+)
- new net SUM4: R48.2, R49.2, U3.3 (+)
