File: docs/v3-adder.kicad_sch (KiCad schematic)
At the start: 101 parts, among them J1 Thonkiconn, J2 Thonkiconn, J3 Thonkiconn, J4 Thonkiconn, J5 Thonkiconn, J6 Thonkiconn, J7 Thonkiconn, J8 Thonkiconn, P1 Eurorack 2x5, SW1A 200-MSP3 (SPDT ON-OFF-ON), SW1B 200-MSP1 (SPDT ON-ON), SW2A 200-MSP3 (SPDT ON-OFF-ON), SW2B 200-MDP6 (DPDT ON-ON-ON), SW3A 200-MSP3 (SPDT ON-OFF-ON), SW3B 200-MDP6 (DPDT ON-ON-ON), SW4A 200-MSP3 (SPDT ON-OFF-ON), SW4B 200-MDP6 (DPDT ON-ON-ON), U1 OPA4196, U2 OPA4196, U3 OPA4196, U4 L78L05, U5 L79L05

Commit message: v3-final
sch complete, panel complete
Other:
- moved on the sheet: C1, C10, C11, C12, C13, C14, C15, C16, C17, C18, C19, C2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

Commit message: component refinement
Parts:
- C11, C12, C13, C14, C15, C16, C17, C18, C19, C2, C20, C4, C5, C6, C7, C8: footprint Capacitor_SMD:C_0805_2012Metric -> Capacitor_SMD:C_1206_3216Metric
- FB1, FB2: footprint 7MM_RESISTOR -> Resistor_THT:R_Axial_DIN0207_L6.3mm_D2.5mm_P7.62mm_Horizontal
- R1, R2, R3, R4: value 50k -> 49.9k; footprint Resistor_SMD:R_0805_2012Metric -> Resistor_SMD:R_1206_3216Metric
- R10, R19, R21, R22, R29, R31, R32, R39, R41, R49: value 1k -> 1.00k; footprint Resistor_SMD:R_0805_2012Metric -> Resistor_SMD:R_1206_3216Metric
- R11, R12: value 12k -> 12.0k; footprint Resistor_SMD:R_0805_2012Metric -> Resistor_SMD:R_1206_3216Metric
- R13: value 5.5k -> 5.49k; footprint Resistor_SMD:R_0805_2012Metric -> Resistor_SMD:R_1206_3216Metric
- R14, R24, R34, R44: footprint Resistor_SMD:R_0805_2012Metric -> Resistor_SMD:R_1206_3216Metric
- R15, R16, R17, R18, R25, R26, R27, R28, R35, R36, R37, R38, R45, R46, R47, R48, R5, R6, R7, R9: value 10k -> 10.0k; footprint Resistor_SMD:R_0805_2012Metric -> Resistor_SMD:R_1206_3216Metric
- R20, R30, R40, R42: value 3k -> 3.00k; footprint Resistor_SMD:R_0805_2012Metric -> Resistor_SMD:R_1206_3216Metric
- R23, R33: value 24.5k -> 24.3k; footprint Resistor_SMD:R_0805_2012Metric -> Resistor_SMD:R_1206_3216Metric
- R43: value 22.5k -> 22.6k; footprint Resistor_SMD:R_0805_2012Metric -> Resistor_SMD:R_1206_3216Metric
- R8: value 20k -> 20.0k; footprint Resistor_SMD:R_0805_2012Metric -> Resistor_SMD:R_1206_3216Metric
- VR1, VR2, VR3, VR4, VR5, VR6: footprint PV36W-MULTITURN-TRIMMER -> Potentiometer_THT:Potentiometer_Bourns_3296W_Vertical
