File: docs/v3-adder.kicad_sch (KiCad schematic)
At the start: 101 parts, among them J1 Thonkiconn, J2 Thonkiconn, J3 Thonkiconn, J4 Thonkiconn, J5 Thonkiconn, J6 Thonkiconn, J7 Thonkiconn, J8 Thonkiconn, P1 Eurorack 2x5, SW1A 200-MSP3 (SPDT ON-OFF-ON), SW1B 200-MSP1 (SPDT ON-ON), SW2A 200-MSP3 (SPDT ON-OFF-ON), SW2B 200-MDP6 (DPDT ON-ON-ON), SW3A 200-MSP3 (SPDT ON-OFF-ON), SW3B 200-MDP6 (DPDT ON-ON-ON), SW4A 200-MSP3 (SPDT ON-OFF-ON), SW4B 200-MDP6 (DPDT ON-ON-ON), U1 OPA4196, U2 OPA4196, U3 OPA4196, U4 L78L05, U5 L79L05

Commit message: changes
Parts:
- J1, J2, J3, J4, J5, J6, J7, J8: footprint THONKICONN-TIGHT -> eurorack:Thonkiconn_PJ301M
- P1: footprint EURO_PWR_HEADER_LOCK -> Connector_IDC:IDC-Header_2x05_P2.54mm_Vertical
- SW1: renamed from SW1A; footprint TAIWAY_200_SP_M2 -> eurorack:SW_Taiway_200_SPDT
- SW2: renamed from SW2A; footprint TAIWAY_200_SP_M2 -> eurorack:SW_Taiway_200_SPDT
- SW3: renamed from SW3A; footprint TAIWAY_200_SP_M2 -> eurorack:SW_Taiway_200_SPDT
- SW4: renamed from SW4A; footprint TAIWAY_200_SP_M2 -> eurorack:SW_Taiway_200_SPDT
- SW5: renamed from SW1B; footprint TAIWAY_200_SP_M2 -> eurorack:SW_Taiway_200_SPDT
- SW6: renamed from SW2B; footprint TAIWAY_200_DP_M2 -> eurorack:SW_Taiway_200_DPDT
- SW7: renamed from SW3B; footprint TAIWAY_200_DP_M2 -> eurorack:SW_Taiway_200_DPDT
- SW8: renamed from SW4B; footprint TAIWAY_200_DP_M2 -> eurorack:SW_Taiway_200_DPDT
Connections:
- net GND: now also J1.S, J1.TN, J2.S, J2.TN, J3.S, J3.TN, J4.S, J5.S, J6.S, J7.S, J8.S; no longer J1.2 (S), J1.3 (N), J2.2 (S), J2.3 (N), J3.2 (S), J3.3 (N), J4.2 (S), J5.2 (S), J6.2 (S), J7.2 (S), J8.2 (S)
- net IN1: now also J1.T; no longer J1.1 (T)
- net IN2: now also J2.T; no longer J2.1 (T)
- net IN3: now also J3.T; no longer J3.1 (T)
- net OUT1_JACK: now also J5.T; no longer J5.1 (T)
- net OUT2_JACK: now also J6.T; no longer J6.1 (T)
- net OUT3_JACK: now also J7.T; no longer J7.1 (T)
- net OUT4_JACK: now also J8.T; no longer J8.1 (T)
- net SUM_JACK: now also J4.T; no longer J4.1 (T)
Changed lines of the file:
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@@
 		(in_pos_files yes)
 		(dnp no)
-		(property "Reference" "SW3B"
+		(property "Reference" "SW7"
 			(at 290.48 145.13 0)
 			(show_name no)
@@
 			)
 		)
-		(property "Footprint" "TAIWAY_200_DP_M2"
+		(property "Footprint" "eurorack:SW_Taiway_200_DPDT"
 			(at 284.48 151.13 0)
 			(hide yes)
@@
 			(project "v3-adder"
 				(path "/8f1c0b1e-0000-4000-8000-000000000001"
-					(reference "SW3B")
+					(reference "SW7")
 					(unit 1)
 				)
@@
 			)
 		)
-		(property "Footprint" "THONKICONN-TIGHT"
+		(property "Footprint" "eurorack:Thonkiconn_PJ301M"
 			(at 147.32 280.67 0)
 			(hide yes)
@@
 			)
 		)
-		(pin "1"
+		(pin "T"
 		)
-		(pin "2"
+		(pin "S"
 		)
 		(instances
@@
 			)
 		)
-		(property "Footprint" "THONKICONN-TIGHT"
+		(property "Footprint" "eurorack:Thonkiconn_PJ301M"
 			(at 411.48 86.36 0)
 			(hide yes)
@@
 			)
 		)
-		(pin "1"
+		(pin "T"
 		)
-		(pin "2"
+		(pin "S"
 		)
-		(pin "3"
+		(pin "TN"
 		)
 		(instances
@@
 			)
 		)
-		(property "Footprint" "THONKICONN-TIGHT"
+		(property "Footprint" "eurorack:Thonkiconn_PJ301M"
 			(at 410.21 114.3 0)
 			(hide yes)
@@
 			)
 		)
-		(pin "1"
+		(pin "T"
 		)
-		(pin "2"
+		(pin "S"
 		)
-		(pin "3"
+		(pin "TN"
 		)
 		(instances
@@
 			)
 		)
-		(property "Footprint" "EURO_PWR_HEADER_LOCK"
+		(property "Footprint" "Connector_IDC:IDC-Header_2x05_P2.54mm_Vertical"
 			(at 387.35 223.52 0)
 			(hide yes)
@@
 		(in_pos_files yes)
 		(dnp no)
-		(property "Reference" "SW2B"
+		(property "Reference" "SW6"
 			(at 291.75 118.46 0)
 			(show_name no)
@@
 			)
 		)
-		(property "Footprint" "TAIWAY_200_DP_M2"
+		(property "Footprint" "eurorack:SW_Taiway_200_DPDT"
 			(at 285.75 124.46 0)
 			(hide yes)
@@
 			(project "v3-adder"
 				(path "/8f1c0b1e-0000-4000-8000-000000000001"
-					(reference "SW2B")
+					(reference "SW6")
 					(unit 1)
 				)
@@
 			)
 		)
-		(property "Footprint" "THONKICONN-TIGHT"
+		(property "Footprint" "eurorack:Thonkiconn_PJ301M"
 			(at 149.86 227.33 0)
 			(hide yes)
@@
 			)
 		)
-		(pin "1"
+		(pin "T"
 		)
-		(pin "2"
+		(pin "S"
 		)
 		(instances
@@
 		(in_pos_files yes)
 		(dnp no)
-		(property "Reference" "SW1B"
+		(property "Reference" "SW5"
 			(at 278.892 84.836 0)
 			(show_name no)
@@
 			)
 		)
-		(property "Footprint" "TAIWAY_200_SP_M2"
+		(property "Footprint" "eurorack:SW_Taiway_200_SPDT"
 			(at 274.32 93.98 0)
 			(hide yes)
@@
 			(project "v3-adder"
 				(path "/8f1c0b1e-0000-4000-8000-000000000001"
-					(reference "SW1B")
+					(reference "SW5")
 					(unit 1)
 				)
@@
 		(in_pos_files yes)
 		(dnp no)
-		(property "Reference" "SW1A"
+		(property "Reference" "SW1"
 			(at 154.94 87.884 0)
 			(show_name no)
@@
 			)
 		)
-		(property "Footprint" "TAIWAY_200_SP_M2"
+		(property "Footprint" "eurorack:SW_Taiway_200_SPDT"
 			(at 154.94 97.79 0)
 			(hide yes)
@@
 			(project "v3-adder"
 				(path "/8f1c0b1e-0000-4000-8000-000000000001"
-					(reference "SW1A")
+					(reference "SW1")
 					(unit 1)
 				)
@@
 		(in_pos_files yes)
 		(dnp no)
-		(property "Reference" "SW4A"
+		(property "Reference" "SW4"
 			(at 151.892 166.37 0)
 			(show_name no)
@@
 			)
 		)
-		(property "Footprint" "TAIWAY_200_SP_M2"
+		(property "Footprint" "eurorack:SW_Taiway_200_SPDT"
 			(at 156.21 176.53 0)
 			(hide yes)
@@
 			(project "v3-adder"
 				(path "/8f1c0b1e-0000-4000-8000-000000000001"
-					(reference "SW4A")
+					(reference "SW4")
 					(unit 1)
 				)
@@
 		(in_pos_files yes)
 		(dnp no)
-		(property "Reference" "SW4B"
+		(property "Reference" "SW8"
 			(at 291.75 183.23 0)
 			(show_name no)
@@
 			)
 		)
-		(property "Footprint" "TAIWAY_200_DP_M2"
+		(property "Footprint" "eurorack:SW_Taiway_200_DPDT"
 			(at 285.75 189.23 0)
 			(hide yes)
@@
 			(project "v3-adder"
 				(path "/8f1c0b1e-0000-4000-8000-000000000001"
-					(reference "SW4B")
+					(reference "SW8")
 					(unit 1)
 				)
@@
 		(in_pos_files yes)
 		(dnp no)
-		(property "Reference" "SW2A"
+		(property "Reference" "SW2"
 			(at 157.226 115.57 0)
 			(show_name no)
@@
 			)
 		)
-		(property "Footprint" "TAIWAY_200_SP_M2"
+		(property "Footprint" "eurorack:SW_Taiway_200_SPDT"
 			(at 157.48 124.46 0)
 			(hide yes)
@@
 			(project "v3-adder"
 				(path "/8f1c0b1e-0000-4000-8000-000000000001"
-					(reference "SW2A")
+					(reference "SW2")
 					(unit 1)
 				)
@@
 			)
 		)
-		(property "Footprint" "THONKICONN-TIGHT"
+		(property "Footprint" "eurorack:Thonkiconn_PJ301M"
 			(at 148.59 300.99 0)
 			(hide yes)
@@
 			)
 		)
-		(pin "1"
+		(pin "T"
 		)
-		(pin "2"
+		(pin "S"
 		)
 		(instances
@@
 		(in_pos_files yes)
 		(dnp no)
-		(property "Reference" "SW3A"
+		(property "Reference" "SW3"
 			(at 152.146 137.668 0)
 			(show_name no)
@@
 			)
 		)
-		(property "Footprint" "TAIWAY_200_SP_M2"
+		(property "Footprint" "eurorack:SW_Taiway_200_SPDT"
 			(at 157.48 148.59 0)
 			(hide yes)
@@
 			(project "v3-adder"
 				(path "/8f1c0b1e-0000-4000-8000-000000000001"
-					(reference "SW3A")
+					(reference "SW3")
 					(unit 1)
 				)
@@
 			)
 		)
-		(property "Footprint" "THONKICONN-TIGHT"
+		(property "Footprint" "eurorack:Thonkiconn_PJ301M"
 			(at 148.59 254 0)
 			(hide yes)
@@
 			)
 		)
-		(pin "1"
+		(pin "T"
 		)
-		(pin "2"
+		(pin "S"
 		)
 		(instances
@@
 			)
 		)
-		(property "Footprint" "THONKICONN-TIGHT"
+		(property "Footprint" "eurorack:Thonkiconn_PJ301M"
 			(at 379.73 138.43 0)
 			(hide yes)
@@
 			)
 		)
-		(pin "1"
+		(pin "T"
 		)
-		(pin "2"
+		(pin "S"
 		)
 		(instances
@@
 			)
 		)
-		(property "Footprint" "THONKICONN-TIGHT"
+		(property "Footprint" "eurorack:Thonkiconn_PJ301M"
 			(at 411.48 101.6 0)
 			(hide yes)
@@
 			)
 		)
-		(pin "1"
+		(pin "T"
 		)
-		(pin "2"
+		(pin "S"
 		)
-		(pin "3"
+		(pin "TN"
 		)
 		(instances

Commit message: Put component values on silk, and write them the same way in both files
Moves all 68 Fab-layer values to the matching silk layer, F.Fab -> F.SilkS
and B.Fab -> B.SilkS so back-side parts keep their mirrored justify. The 20
values that were already hidden stay hidden: "200-MDP6 (DPDT ON-ON-ON)" has
nowhere to go on a 19.6 mm board.

Trailing zeros that carry no information go with them -- 10.0k reads 10k,
1.00k reads 1k -- while 49.9k, 24.3k, 22.6k, 5.49k and 619R keep every
digit. Tolerance was never legible at 4 HP anyway; it lives in the BOM.

This turned out to be a consistency fix rather than a cosmetic one. The
schematic was the clean side: all ten 1k parts read 1.00k there and all
twenty 10k read 10.0k, but three of them had been edited to 1k in pcbnew,
and R8 disagreed outright (20.0k against the board's 20k). R31 read 1.00k
beside R32's 1k in the same ladder; R30 read 3.00k while R40, its exact
peer one stage along, read 3k. All 101 references now match between
schematic and board, with the netlist node-for-node identical to before
the edit and ERC still at zero.

gen_schematic.py moves in lockstep -- both the emitted values and the
check_function comparison strings, or --check would start failing. The E24
rationale comment keeps its decimals, since the argument turns on 3.01k
against 3.00k.

The BOM's "changes from what is currently in the schematic" table now reads
backwards for its first two rows, so it gets a note rather than a rewrite:
the parts did not change back, only the label got shorter.

Also carries the routing done in the meantime: 511 -> 677 segments, 98 more
vias, and no unconnected items left.
Parts:
- R10, R19, R21, R22, R29, R31, R32, R39, R41, R49: value 1.00k -> 1k
- R11, R12: value 12.0k -> 12k
- R15, R16, R17, R18, R25, R26, R27, R28, R35, R36, R37, R38, R45, R46, R47, R48, R5, R6, R7, R9: value 10.0k -> 10k
- R20, R30, R40, R42: value 3.00k -> 3k
- R8: value 20.0k -> 20k
Changed lines of the file:
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@@
 			)
 		)
-		(property "Value" "1.00k"
+		(property "Value" "1k"
 			(at 176.53 300.736 0)
 			(show_name no)
@@
 			)
 		)
-		(property "Value" "1.00k"
+		(property "Value" "1k"
 			(at 208.74 154.59 0)
 			(show_name no)
@@
 			)
 		)
-		(property "Value" "10.0k"
+		(property "Value" "10k"
 			(at 188.77 236.57 0)
 			(show_name no)
@@
 			)
 		)
-		(property "Value" "10.0k"
+		(property "Value" "10k"
 			(at 190.5 279.654 0)
 			(show_name no)
@@
 			)
 		)
-		(property "Value" "10.0k"
+		(property "Value" "10k"
 			(at 210.01 223.17 0)
 			(show_name no)
@@
 			)
 		)
-		(property "Value" "10.0k"
+		(property "Value" "10k"
 			(at 207.264 300.482 0)
 			(show_name no)
@@
 			)
 		)
-		(property "Value" "12.0k"
+		(property "Value" "12k"
 			(at 221.44 103.79 0)
 			(show_name no)
@@
 			)
 		)
-		(property "Value" "20.0k"
+		(property "Value" "20k"
 			(at 402.13 136.24 0)
 			(show_name no)
@@
 			)
 		)
-		(property "Value" "10.0k"
+		(property "Value" "10k"
 			(at 207.47 275.24 0)
 			(show_name no)
@@
 			)
 		)
-		(property "Value" "10.0k"
+		(property "Value" "10k"
 			(at 205.486 279.654 0)
 			(show_name no)
@@
 			)
 		)
-		(property "Value" "3.00k"
+		(property "Value" "3k"
 			(at 239.22 130.46 0)
 			(show_name no)
@@
 			)
 		)
-		(property "Value" "10.0k"
+		(property "Value" "10k"
 			(at 207.01 253.238 0)
 			(show_name no)
@@
 			)
 		)
-		(property "Value" "10.0k"
+		(property "Value" "10k"
 			(at 424.64 173.64 0)
 			(show_name no)
@@
 			)
 		)
-		(property "Value" "10.0k"
+		(property "Value" "10k"
 			(at 403.4 161.64 0)
 			(show_name no)
@@
 			)
 		)
-		(property "Value" "10.0k"
+		(property "Value" "10k"
 			(at 208.026 226.314 0)
 			(show_name no)
@@
 			)
 		)
-		(property "Value" "1.00k"
+		(property "Value" "1k"
 			(at 208.74 130.46 0)
 			(show_name no)
@@
 			)
 		)
-		(property "Value" "10.0k"
+		(property "Value" "10k"
 			(at 417.37 136.24 0)
 			(show_name no)
@@
 			)
 		)
-		(property "Value" "1.00k"
+		(property "Value" "1k"
 			(at 223.98 154.59 0)
 			(show_name no)
@@
 			)
 		)
-		(property "Value" "12.0k"
+		(property "Value" "12k"
 			(at 206.2 103.79 0)
 			(show_name no)
@@
 			)
 		)
-		(property "Value" "10.0k"
+		(property "Value" "10k"
 			(at 210.01 248.57 0)
 			(show_name no)
@@
 			)
 		)
-		(property "Value" "10.0k"
+		(property "Value" "10k"
 			(at 192.532 226.06 0)
 			(show_name no)
@@
 			)
 		)
-		(property "Value" "10.0k"
+		(property "Value" "10k"
 			(at 389.08 105.06 0)
 			(show_name no)
@@
 			)
 		)
-		(property "Value" "10.0k"
+		(property "Value" "10k"
 			(at 191.516 252.73 0)
 			(show_name no)
@@
 			)
 		)
-		(property "Value" "1.00k"
+		(property "Value" "1k"
 			(at 225.25 182.53 0)
 			(show_name no)
@@
 			)
 		)
-		(property "Value" "10.0k"
+		(property "Value" "10k"
 			(at 186.23 263.24 0)
 			(show_name no)
@@
 			)
 		)
-		(property "Value" "10.0k"
+		(property "Value" "10k"
 			(at 188.77 211.17 0)
 			(show_name no)
@@
 			)
 		)
-		(property "Value" "10.0k"
+		(property "Value" "10k"
 			(at 389.08 117.76 0)
 			(show_name no)
@@
 			)
 		)
-		(property "Value" "3.00k"
+		(property "Value" "3k"
 			(at 239.22 154.59 0)
 			(show_name no)
@@
 			)
 		)
-		(property "Value" "1.00k"
+		(property "Value" "1k"
 			(at 177.8 226.06 0)
 			(show_name no)
@@
 			)
 		)
-		(property "Value" "1.00k"
+		(property "Value" "1k"
 			(at 175.768 280.162 0)
 			(show_name no)
@@
 			)
 		)
-		(property "Value" "10.0k"
+		(property "Value" "10k"
 			(at 192.278 299.974 0)
 			(show_name no)
@@
 			)
 		)
-		(property "Value" "1.00k"
+		(property "Value" "1k"
 			(at 176.276 252.222 0)
 			(show_name no)
@@
 			)
 		)
-		(property "Value" "10.0k"
+		(property "Value" "10k"
 			(at 389.08 89.82 0)
 			(show_name no)
@@
 			)
 		)
-		(property "Value" "3.00k"
+		(property "Value" "3k"
 			(at 210.01 182.53 0)
 			(show_name no)
@@
 			)
 		)
-		(property "Value" "3.00k"
+		(property "Value" "3k"
 			(at 240.49 182.53 0)
 			(show_name no)
@@
 			)
 		)
-		(property "Value" "1.00k"
+		(property "Value" "1k"
 			(at 389.08 159.67 0)
 			(show_name no)
@@
 			)
 		)
-		(property "Value" "1.00k"
+		(property "Value" "1k"
 			(at 223.98 130.46 0)
 			(show_name no)

Commit message: Put the board-to-board connectors in the schematic
The eight interconnect footprints existed only on the board, carrying REF** and
absent from the schematic entirely. Update PCB from Schematic would have offered
to delete them, they were missing from the BOM, and nothing checked their pin
mapping -- it was correct, but only because it had been checked by hand.

Adds adder:HDR1x6 to the symbol library and eight instances: P2-P5 are the pin
headers on the control board's rear, P6-P9 the sockets on the trimmer board's
front, each Value naming the part it mates with. Board footprints annotated to
match. The five spare pins per side are carried as no-connects so they stay
available rather than becoming ERC noise.

Two things caught by checks rather than by care. Placing on a round 1 mm grid
put every pin off KiCad's 1.27 connection grid -- 46 warnings; coordinates are
now multiples of 1.27. Worse, the first placement dropped the row onto a wire at
y=344.17 and silently merged OUT4, S2_4th, REFN_TOP and REFN_W into one net.
ERC called it a naming conflict rather than a short, and the free-space check
that cleared the area had only looked at symbol and label anchors -- it never
read wire geometry, so it could not have seen the wire it collided with. The
placement now rasterises wires, symbols and labels together and asserts each
target box is clear before writing.

ERC 0 violations. DRC 0 errors, 0 unconnected. 109 references on both sides with
no orphans and no value or footprint mismatch. Netlist diff against the
pre-edit sheet: 48 connector pins added, 0 other nets changed.
Parts:
- added P2: 1x6 pin header (mates P6), Connector_PinHeader_2.54mm:PinHeader_1x06_P2.54mm_Vertical, symbol adder:HDR1x6
- added P3: 1x6 pin header (mates P7), Connector_PinHeader_2.54mm:PinHeader_1x06_P2.54mm_Vertical, symbol adder:HDR1x6
- added P4: 1x6 pin header (mates P8), Connector_PinHeader_2.54mm:PinHeader_1x06_P2.54mm_Vertical, symbol adder:HDR1x6
- added P5: 1x6 pin header (mates P9), Connector_PinHeader_2.54mm:PinHeader_1x06_P2.54mm_Vertical, symbol adder:HDR1x6
- added P6: 1x6 socket (mates P2), Connector_PinSocket_2.54mm:PinSocket_1x06_P2.54mm_Vertical, symbol adder:HDR1x6
- added P7: 1x6 socket (mates P3), Connector_PinSocket_2.54mm:PinSocket_1x06_P2.54mm_Vertical, symbol adder:HDR1x6
- added P8: 1x6 socket (mates P4), Connector_PinSocket_2.54mm:PinSocket_1x06_P2.54mm_Vertical, symbol adder:HDR1x6
- added P9: 1x6 socket (mates P5), Connector_PinSocket_2.54mm:PinSocket_1x06_P2.54mm_Vertical, symbol adder:HDR1x6
Connections:
- net +12V: now also P2.6 (P6), P4.1 (P1), P6.6 (P6), P8.1 (P1)
- net -12V: now also P3.6 (P6), P7.6 (P6)
- net GND: now also P2.1 (P1), P3.1 (P1), P4.6 (P6), P5.6 (P6), P6.1 (P1), P7.1 (P1), P8.6 (P6), P9.6 (P6)
- net LAD1_TOP: now also P3.2 (P2), P7.2 (P2)
- net LAD1_TRIM: now also P3.5 (P5), P7.5 (P5)
- net LAD2_TOP: now also P3.3 (P3), P7.3 (P3)
- net LAD3_TOP: now also P4.5 (P5), P8.5 (P5)
- net LAD4_TOP: now also P5.3 (P3), P9.3 (P3)
- net REFN_TOP: now also P4.4 (P4), P8.4 (P4)
- net REFN_W: now also P5.4 (P4), P9.4 (P4)
- net REFP_TOP: now also P2.2 (P2), P6.2 (P2)
- net REFP_W: now also P4.2 (P2), P8.2 (P2)
- net S2_4th: now also P3.4 (P4), P7.4 (P4)
- net S3_4th: now also P5.2 (P2), P9.2 (P2)
- net S4_5th: now also P5.1 (P1), P9.1 (P1)
- no-connect marks 0 -> 10
